File: boards/wt-keyer.kicad_pcb (KiCad board)
At the start: 2 copper layers, 90 x 70 mm, 61 parts, among them IC1 ATmega8A-P, J2 Paddle, J3 Speaker, J4 Walkie-Talkie, J5 Power 5V, Q1 2N 3904, SW1 Cmd, SW2 Pitch, SW3 WPM, U1 LM386-1

Commit message: Updated the files for V2 of the walkie-talkie keyer.
Parts:
- added C22: 10nF, Capacitor_THT:C_Disc_D3.0mm_W1.6mm_P2.50mm, F.Cu at (112.7, 120.7)
- added FB8: Ferrite Bead, Inductor_THT:L_Axial_L9.5mm_D4.0mm_P2.54mm_Vertical_Fastron_SMCC, F.Cu at (119.8, 93.7)
- added J5: Headphones, Connector_Audio:Jack_3.5mm_Ledino_KB3SPRS_Horizontal, F.Cu at (107.8, 112.9)
- added J6: USB-C, Connector_USB:USB_C_Receptacle_GCT_USB4125-xx-x-0190_6P_TopMnt_Horizontal, F.Cu at (105.4, 121.6)
- added R15: 10kΩ, Resistor_THT:R_Axial_DIN0207_L6.3mm_D2.5mm_P2.54mm_Vertical, F.Cu at (112.7, 123.5)
- added REF**: Hole_5mm_No_Courtyard, footprints:Hole_5mm_No_Courtyard, F.Cu at (166.5, 138.0)
- added REF**: Hole_5mm_No_Courtyard, footprints:Hole_5mm_No_Courtyard, F.Cu at (166.5, 105.0)
- C13, C18, C21: footprint Capacitor_THT:CP_Radial_D6.3mm_P2.50mm -> Capacitor_THT:CP_Radial_D5.0mm_P2.50mm
- H1, H2, H3, H4: footprint MountingHole:MountingHole_3.2mm_M3_ISO7380_Pad_TopBottom -> footprints:MountingHole_3.2mm_M3_Pad_5.0mm_TopBottom
- IC1: footprint Package_DIP:DIP-28_W7.62mm_Socket_LongPads -> Package_DIP:DIP-28_W7.62mm
- J1: renamed from J5; footprint Connector_PinSocket_2.54mm:PinSocket_1x02_P2.54mm_Vertical -> footprints:FanPinHeader_1x02_P2.54mm_Vertical
- J4: footprint footprints:DIN_5Pin_Horizontal -> footprints:DIN_7Pin_Horizontal
- P1: renamed from Vol1; value 10kΩ log -> 10kΩ lin
- Q1: value 2N 3904 -> 2N3904; footprint Package_TO_SOT_THT:TO-92_Inline_Wide -> Package_TO_SOT_THT:TO-92_Inline
- R8: value 100kΩ -> 47kΩ
- RV1, RV2: moved to F.Cu
- SW1: value Cmd -> C
- SW2: value Pitch -> 1
- SW3: value WPM -> 2
- moved RV1 14.0 mm to (169.2, 143.0)
- moved FB6 13.1 mm to (119.8, 98.3)
- moved C14 9.56 mm to (115.0, 138.6), turned to 90 degrees
- moved Q1 8.49 mm to (154.7, 129.6), turned to 90 degrees
- moved C16 8.48 mm to (148.6, 87.6)
- moved J2 6.95 mm to (171.3, 85.6), turned to 180 degrees
- moved R11 6.91 mm to (146.9, 129.6), turned to 90 degrees
- moved FB5 6.87 mm to (116.8, 83.7)
- moved C20 6.65 mm to (158.9, 124.5)
- moved R3 6.08 mm to (150.3, 122.1), turned to 90 degrees
- moved FB7 5.65 mm to (119.8, 89.1)
- moved RV2 5.36 mm to (169.2, 110.0)
- moved R8 4.49 mm to (131.2, 143.5)
- moved R9 4.38 mm to (162.0, 127.5), turned to -90 degrees
- moved C6 3.80 mm to (151.1, 116.2)
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- renumbered U1 to IC2, J3 to J2, J2 to J3
Connections:
- C18 pad 2: Net-(J3-Pin_3) -> Net-(C18-Pad2)
- J2 pad 3: Net-(J3-Pin_3) -> Net-(J2-Pin_3)
- Q1 pad 1: Net-(Q1-C) -> GND
- Q1 pad 3: GND -> Net-(Q1-C)
Routing:
- net GND: track 387.6 -> 502.4 mm
- net Net-(J2-Pin_3): track 0.00 -> 82.2 mm
- net Net-(C18-Pad2): track 0.00 -> 40.9 mm
- net Net-(FB8-Pad1): track 0.00 -> 25.0 mm
- net Net-(Conn1-Pin_2): track 99.4 -> 124.3 mm
- net Net-(IC1-PD0): track 31.0 -> 12.9 mm
- net Net-(IC2-+): track 82.9 -> 65.4 mm
- net Net-(J3-Pin_3): track 15.1 -> 0.00 mm
- net Net-(J6-CC1): track 0.00 -> 12.2 mm
- net Net-(IC1-PD7): track 45.7 -> 35.7 mm
- net Net-(FB6-Pad1): track 4.60 -> 13.4 mm
- net Net-(IC1-PD1): track 17.6 -> 25.7 mm
- net Net-(Q1-C): track 21.3 -> 15.0 mm
- net Net-(C15-Pad2): track 12.8 -> 7.64 mm
- net Net-(R14-Pad1): track 27.0 -> 23.3 mm
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Other:
- board text added: "Walkie-Talkie Keyer V2 by DF5WC 2025"
- board text removed: "Walkie-Talkie Keyer V1 by DF5WC 2025"
