File: boards/wt-keyer.kicad_sch (KiCad schematic)
At the start: 62 parts, among them IC1 ATmega8A-P, J2 Paddle, J3 Speaker, J4 Walkie-Talkie, J5 Power 5V, Q1 2N 3904, SW1 Cmd, SW2 Pitch, SW3 WPM, U1 LM386-1

Commit message: Updated the files for V2 of the walkie-talkie keyer.
Parts:
- removed J4: Walkie-Talkie, footprints:DIN_5Pin_Horizontal, symbol Connector:DIN-5_180degree
- removed LS1: Speaker 8Ω, symbol Device:Speaker
- removed Q1: 2N 3904, Package_TO_SOT_THT:TO-92_Inline_Wide, symbol Transistor_BJT:BC237
- added C22: 10nF, Capacitor_THT:C_Disc_D3.0mm_W1.6mm_P2.50mm, symbol Device:C_Small
- added FB8: Ferrite Bead, Inductor_THT:L_Axial_L9.5mm_D4.0mm_P2.54mm_Vertical_Fastron_SMCC, symbol Device:FerriteBead_Small
- added J4: Walkie-Talkie, footprints:DIN_7Pin_Horizontal, symbol Connector:DIN-7
- added J5: Headphones, Connector_Audio:Jack_3.5mm_Ledino_KB3SPRS_Horizontal, symbol Connector_Audio:AudioJack3_SwitchTR
- added J6: USB-C, Connector_USB:USB_C_Receptacle_GCT_USB4125-xx-x-0190_6P_TopMnt_Horizontal, symbol Connector:USB_C_Receptacle_PowerOnly_6P
- added Q1: 2N3904, Package_TO_SOT_THT:TO-92_Inline, symbol Transistor_BJT:2N3904
- added R15: 10kΩ, Resistor_THT:R_Axial_DIN0207_L6.3mm_D2.5mm_P2.54mm_Vertical, symbol Device:R_Small
- C13, C18, C21: footprint Capacitor_THT:CP_Radial_D6.3mm_P2.50mm -> Capacitor_THT:CP_Radial_D5.0mm_P2.50mm
- H1, H2, H3, H4: footprint MountingHole:MountingHole_3.2mm_M3_ISO7380_Pad_TopBottom -> footprints:MountingHole_3.2mm_M3_Pad_5.0mm_TopBottom
- IC1: footprint Package_DIP:DIP-28_W7.62mm_Socket_LongPads -> Package_DIP:DIP-28_W7.62mm
- J1: renamed from J5; footprint Connector_PinSocket_2.54mm:PinSocket_1x02_P2.54mm_Vertical -> footprints:FanPinHeader_1x02_P2.54mm_Vertical
- P1: renamed from Vol1; value 10kΩ log -> 10kΩ lin
- R8: value 33kΩ -> 47kΩ
- SW1: value Cmd -> C
- SW2: value Pitch -> 1
- SW3: value WPM -> 2
- renumbered U1 to IC2, J3 to J2, J2 to J3
Connections:
- net GND: now also C22.2, J5.S, J6.A12 (GND), J6.B12 (GND), J6.S1 (SHIELD), Q1.1 (E), R15.1
- net at C13.1, C16.1, C3.1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: now also C22.1, J6.A9 (VBUS), J6.B9 (VBUS)
- net at FB2.1: now also J4.1
- net at FB3.1: now also J4.2
- net at C18.2: now also FB8.2; no longer J2.3 (Pin_3)
- net at R10.2, R11.2: now also Q1.2 (B)
- net at C20.1, FB1.2: now also Q1.3 (C)
- net at FB4.1: now also J4.3
- net at FB1.1: now also J4.4
- new net: J6.A5 (CC1), R15.2
- new net: FB8.1, J5.R, J5.T
- new net: J2.3 (Pin_3), J5.RN, J5.TN
- no-connect marks 17 -> 18
Other:
- added sheet Supplementary (wt-keyer-supplementary.kicad_sch)
- moved on the sheet: C1, C10, C11, C12, C13, C14, C15, C16, C17, C18, C19, C2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
